Commit message: updated arachne urdf

File: robots/arachne/arachne.urdf (robot description, URDF)
Before this commit: robot arachne, 19 links, 18 joints
Links:
- removed link femur
- removed link femur_2
- removed link femur_3
- removed link femur_4
- removed link femur_5
- removed link femur_6
- removed link hip
- removed link hip_2
- removed link hip_3
- removed link hip_4
- removed link hip_5
- removed link hip_6
- added link rightfemur, mass 0.0986065; collision mesh filename=package://assets/e07_mg996r.stl; collision mesh filename=package://assets/idler.stl
- added link rightfemur_2, mass 0.0986065; collision mesh filename=package://assets/e07_mg996r.stl; collision mesh filename=package://assets/idler.stl
- added link rightfemur_3, mass 0.0986065; collision mesh filename=package://assets/e07_mg996r.stl; collision mesh filename=package://assets/idler.stl
- added link rightfemur_4, mass 0.0986065; collision mesh filename=package://assets/e07_mg996r.stl; collision mesh filename=package://assets/idler.stl
- added link rightfemur_5, mass 0.0986065; collision mesh filename=package://assets/e07_mg996r.stl; collision mesh filename=package://assets/idler.stl
- added link rightfemur_6, mass 0.0986065; collision mesh filename=package://assets/e07_mg996r.stl; collision mesh filename=package://assets/idler.stl
- added link righthip, mass 0.0839378; collision mesh filename=package://assets/e07_mg996r.stl; collision mesh filename=package://assets/idler.stl
- added link righthip_2, mass 0.0839378; collision mesh filename=package://assets/e07_mg996r.stl; collision mesh filename=package://assets/idler.stl
- added link righthip_3, mass 0.0839378; collision mesh filename=package://assets/e07_mg996r.stl; collision mesh filename=package://assets/idler.stl
- added link righthip_4, mass 0.0839378; collision mesh filename=package://assets/e07_mg996r.stl; collision mesh filename=package://assets/idler.stl
- added link righthip_5, mass 0.0839378; collision mesh filename=package://assets/e07_mg996r.stl; collision mesh filename=package://assets/idler.stl
- added link righthip_6, mass 0.0839378; collision mesh filename=package://assets/e07_mg996r.stl; collision mesh filename=package://assets/idler.stl
- link lowerbody: mass 0.776148 -> 1.10838; geometry collision mesh filename=package://assets/e07_mg996r.stl; collision mesh filename=package://assets/e07_mg996r.stl
- link tibia: mass 0.0478411 -> 0.0352344
- link tibia_2: mass 0.0478411 -> 0.0352344
- link tibia_3: mass 0.0478411 -> 0.0352344
- link tibia_4: mass 0.0478411 -> 0.0352344
- link tibia_5: mass 0.0478411 -> 0.0352344
- link tibia_6: mass 0.0478411 -> 0.0352344
Joints:
- joint femur_l1: child femur_4 -> rightfemur_4; origin xyz=0.13 -2.77556e-17 -3.1225e-17 rpy=-3.14159 1.19807e-14 2.53073 -> xyz=0.085 -1.38778e-17 0 rpy=-3.14159 1.18794e-14 2.53073
- joint femur_l2: child femur_5 -> rightfemur_5; origin xyz=0.13 0 3.46945e-17 rpy=3.14159 8.05484e-15 2.53073 -> xyz=0.085 -2.77556e-17 -9.51402e-18 rpy=3.14159 8.05484e-15 2.53073
- joint femur_l3: child femur_6 -> rightfemur_6; limit lower=-2.18166 upper=5.77316e-15 effort=10 velocity=6 -> lower=-2.18166 upper=5.32907e-15 effort=10 velocity=6; origin xyz=0.13 0 0 rpy=3.14159 6.7833e-16 2.53073 -> xyz=0.085 0 0 rpy=3.14159 -3.33067e-16 2.53073
- joint femur_r1: child femur -> rightfemur; origin xyz=-0.12216 -0.0444626 -3.45557e-15 rpy=-3.14159 1.8554e-14 0.959931 -> xyz=-0.0798739 -0.0290717 -2.22045e-15 rpy=-3.14159 1.84852e-14 0.959931
- joint femur_r2: child femur_2 -> rightfemur_2; origin xyz=-0.12216 -0.0444626 -1.38778e-17 rpy=-3.14159 1.60405e-14 0.959931 -> xyz=-0.0798739 -0.0290717 -3.23092e-17 rpy=-3.14159 1.60384e-14 0.959931
- joint femur_r3: child femur_3 -> rightfemur_3; origin xyz=-0.12216 -0.0444626 8.60423e-16 rpy=3.14159 -1.93599e-14 0.959931 -> xyz=-0.0798739 -0.0290717 6.17562e-16 rpy=3.14159 -1.93734e-14 0.959931
- joint hip_l1: child hip_4 -> righthip_4; limit lower=-0.523599 upper=0.523599 effort=10 velocity=6 -> lower=-0.533126 upper=0.514071 effort=10 velocity=6; origin xyz=-0.134145 -0.107445 0.00709854 rpy=3.14159 5.2737e-16 0.668693 -> xyz=-0.129135 -0.119156 0.0319385 rpy=3.14159 7.46399e-15 0.678221
- joint hip_l2: child hip_5 -> righthip_5; origin xyz=-0.140028 -0.0156824 0.00709854 rpy=-3.14159 -1.75355e-16 -8.38581e-15 -> xyz=-0.131169 -0.0202089 0.0319385 rpy=-3.14159 -1.75355e-16 -4.49293e-15
- joint hip_l3: child hip_6 -> righthip_6; origin xyz=-0.138347 0.0804306 0.00709854 rpy=-3.14159 7.69581e-15 -0.436332 -> xyz=-0.125258 0.0663725 0.0319385 rpy=3.14159 3.08664e-15 -0.436332
- joint hip_r1: child hip -> righthip; origin xyz=0.0252111 -0.108204 0.00709854 rpy=3.14159 3.08939e-15 2.46337 -> xyz=0.052388 -0.119156 0.0319385 rpy=3.14159 9.93205e-15 2.46337
- joint hip_r2: child hip_2 -> righthip_2; limit lower=-0.523599 upper=0.523599 effort=10 velocity=6 -> lower=-0.533126 upper=0.514071 effort=10 velocity=6; origin xyz=0.0319685 -0.0165017 0.00709854 rpy=3.14159 -3.06292e-15 3.13207 -> xyz=0.054422 -0.0202089 0.0319385 rpy=3.14159 -3.06367e-15 3.14159
- joint hip_r3: child hip_3 -> righthip_3; limit lower=-0.523599 upper=0.523599 effort=10 velocity=6 -> lower=-0.533126 upper=0.514071 effort=10 velocity=6; origin xyz=0.0312028 0.0796229 0.00709854 rpy=3.14159 2.09797e-15 -2.71479 -> xyz=0.0485111 0.0663725 0.0319385 rpy=-3.14159 -2.57421e-15 -2.70526
- joint tibia_l1: limit lower=-1.22173 upper=0 effort=10 velocity=6 -> lower=-1.22173 upper=1.11022e-15 effort=10 velocity=6; origin xyz=-0.0627954 0.0234 0.0095 rpy=-1.5708 1.22173 -3.14159 -> xyz=-0.0532205 0.022894 0.0149 rpy=-1.5708 1.22173 -3.13207; parent hip_4 -> righthip_4
- joint tibia_l2: origin xyz=-0.0627954 0.0234 0.0095 rpy=-1.5708 1.22173 -3.14159 -> xyz=-0.053 0.0234 0.0149 rpy=-1.5708 1.22173 -3.14159; parent hip_5 -> righthip_5
- joint tibia_l3: limit lower=-1.22173 upper=7.99361e-15 effort=10 velocity=6 -> lower=-1.22173 upper=2.66454e-15 effort=10 velocity=6; origin xyz=-0.0627954 0.0234 0.0095 rpy=-1.5708 1.22173 3.14159 -> xyz=-0.053 0.0234 0.0149 rpy=-1.5708 1.22173 3.14159; parent hip_6 -> righthip_6
- joint tibia_r1: limit lower=-2.22045e-15 upper=1.22173 effort=10 velocity=6 -> lower=-8.43769e-15 upper=1.22173 effort=10 velocity=6; origin xyz=-0.0697954 -0.0234 0.0115 rpy=-1.5708 -1.5708 0 -> xyz=-0.06 -0.0234 0.0146 rpy=-1.5708 -1.5708 0; parent hip -> righthip
- joint tibia_r2: origin xyz=-0.0697954 -0.0234 0.0115 rpy=-1.5708 -1.5708 0 -> xyz=-0.0597743 -0.0239706 0.0146 rpy=-1.56127 -1.5708 0; parent hip_2 -> righthip_2
- joint tibia_r3: limit lower=-2.35367e-14 upper=1.22173 effort=10 velocity=6 -> lower=-1.82077e-14 upper=1.22173 effort=10 velocity=6; origin xyz=-0.0697954 -0.0234 0.0115 rpy=-1.5708 -1.5708 0 -> xyz=-0.0597743 -0.0239706 0.0146 rpy=-1.56127 -1.5708 0; parent hip_3 -> righthip_3

Commit message: updated urdf, argparser functionality

File: robots/arachne/arachne.urdf (robot description, URDF)
Before this commit: robot arachne, 19 links, 18 joints
Joints:
- joint femur_l1: limit lower=-2.18166 upper=0 effort=10 velocity=6 -> lower=-0.959931 upper=1.22173 effort=10 velocity=6; origin xyz=0.085 -1.38778e-17 0 rpy=-3.14159 1.18794e-14 2.53073 -> xyz=0.085 -3.46945e-18 -2.77556e-17 rpy=-3.14159 1.11022e-16 -2.53073
- joint femur_l2: limit lower=-2.18166 upper=0 effort=10 velocity=6 -> lower=-0.959931 upper=1.22173 effort=10 velocity=6; origin xyz=0.085 -2.77556e-17 -9.51402e-18 rpy=3.14159 8.05484e-15 2.53073 -> xyz=0.085 3.46945e-18 -7.99785e-18 rpy=-3.14159 6.12323e-17 -2.53073
- joint femur_l3: limit lower=-2.18166 upper=5.32907e-15 effort=10 velocity=6 -> lower=-0.959931 upper=1.22173 effort=10 velocity=6; origin xyz=0.085 0 0 rpy=3.14159 -3.33067e-16 2.53073 -> xyz=0.085 -2.80678e-15 1.76248e-15 rpy=3.14159 1.4988e-15 -2.53073
- joint femur_r1: limit lower=-1.5099e-14 upper=2.18166 effort=10 velocity=6 -> lower=-1.22173 upper=0.959931 effort=10 velocity=6; origin xyz=-0.0798739 -0.0290717 -2.22045e-15 rpy=-3.14159 1.84852e-14 0.959931 -> xyz=-3.1225e-17 -0.085 0 rpy=3.14159 -5.55112e-17 0.959931
- joint femur_r2: limit lower=0 upper=2.18166 effort=10 velocity=6 -> lower=-1.22173 upper=0.959931 effort=10 velocity=6; origin xyz=-0.0798739 -0.0290717 -3.23092e-17 rpy=-3.14159 1.60384e-14 0.959931 -> xyz=1.63064e-16 -0.085 -1.75641e-17 rpy=-3.14159 3.72966e-17 0.959931
- joint femur_r3: limit lower=0 upper=2.18166 effort=10 velocity=6 -> lower=-1.22173 upper=0.959931 effort=10 velocity=6; origin xyz=-0.0798739 -0.0290717 6.17562e-16 rpy=3.14159 -1.93734e-14 0.959931 -> xyz=-1.9082e-16 -0.085 -2.77556e-17 rpy=-3.14159 2.22045e-16 0.959931
- joint tibia_l1: limit lower=-1.22173 upper=1.11022e-15 effort=10 velocity=6 -> lower=0 upper=1.22173 effort=10 velocity=6; origin xyz=-0.0532205 0.022894 0.0149 rpy=-1.5708 1.22173 -3.13207 -> xyz=-0.0532205 0.022894 0.0149 rpy=-1.5708 -7.54732e-15 -3.13207
- joint tibia_l2: limit lower=-1.22173 upper=1.11022e-15 effort=10 velocity=6 -> lower=0 upper=1.22173 effort=10 velocity=6; origin xyz=-0.053 0.0234 0.0149 rpy=-1.5708 1.22173 -3.14159 -> xyz=-0.053 0.0234 0.0149 rpy=-1.5708 8.66856e-15 3.14159
- joint tibia_l3: limit lower=-1.22173 upper=2.66454e-15 effort=10 velocity=6 -> lower=0 upper=1.22173 effort=10 velocity=6; origin xyz=-0.053 0.0234 0.0149 rpy=-1.5708 1.22173 3.14159 -> xyz=-0.053 0.0234 0.0149 rpy=-1.5708 7.74969e-17 3.14159
- joint tibia_r1: limit lower=-8.43769e-15 upper=1.22173 effort=10 velocity=6 -> lower=-1.22173 upper=1.06581e-14 effort=10 velocity=6
- joint tibia_r2: limit lower=0 upper=1.22173 effort=10 velocity=6 -> lower=-1.22173 upper=3.81917e-14 effort=10 velocity=6
- joint tibia_r3: limit lower=-1.82077e-14 upper=1.22173 effort=10 velocity=6 -> lower=-1.22173 upper=7.99361e-15 effort=10 velocity=6
